Commit message: fix bugs in dreamwaq training; improve policy export; genesis still exists bugs

File: resources/robots/go2/urdf/go2.urdf (robot description, URDF)
Before this commit: robot go2_description, 29 links, 28 joints
Links:
- link FL_calf: geometry collision cylinder length=0.12 radius=0.013; visual mesh filename=../dae/calf.dae
- link FL_hip: geometry collision cylinder length=0.12 radius=0.04; visual mesh filename=../dae/hip.dae
- link FL_thigh: geometry collision box size=0.2 0.0245 0.034; visual mesh filename=../dae/thigh.dae
- link FR_hip: geometry collision cylinder length=0.12 radius=0.04; visual mesh filename=../dae/hip.dae
- link FR_thigh: geometry collision box size=0.2 0.0245 0.034; visual mesh filename=../dae/thigh_mirror.dae
- link RL_hip: geometry collision cylinder length=0.12 radius=0.046; visual mesh filename=../dae/hip.dae
- link RL_thigh: geometry collision box size=0.2 0.0245 0.034; visual mesh filename=../dae/thigh.dae
- link RR_hip: geometry collision cylinder length=0.12 radius=0.046; visual mesh filename=../dae/hip.dae
- link RR_thigh: geometry collision box size=0.2 0.0245 0.034; visual mesh filename=../dae/thigh_mirror.dae
- link base: geometry collision box size=0.26 0.18 0.15; visual mesh filename=../dae/base.dae

Commit message: fix bugs in genesis training

File: resources/robots/go2/urdf/go2.urdf (robot description, URDF)
Before this commit: robot go2_description, 29 links, 28 joints
Links:
- added link FL_calf_rotor, mass 0.089
- added link FL_hip_rotor, mass 0.089
- added link FL_thigh_rotor, mass 0.089
- added link FR_calf_rotor, mass 0.089
- added link FR_hip_rotor, mass 0.089
- added link FR_thigh_rotor, mass 0.089
- added link RL_calf_rotor, mass 0.089
- added link RL_hip_rotor, mass 0.089
- added link RL_thigh_rotor, mass 0.089
- added link RR_calf_rotor, mass 0.089
- added link RR_hip_rotor, mass 0.089
- added link RR_thigh_rotor, mass 0.089
- added link front_camera
- link FL_calf: geometry collision cylinder length=0.12 radius=0.012; visual mesh filename=../dae/calf.dae
- link FL_hip: geometry collision cylinder length=0.04 radius=0.046; visual mesh filename=../dae/hip.dae
- link FL_thigh: geometry collision box size=0.213 0.0245 0.034; visual mesh filename=../dae/thigh.dae
- link FR_hip: geometry collision cylinder length=0.04 radius=0.046; visual mesh filename=../dae/hip.dae
- link FR_thigh: geometry collision box size=0.213 0.0245 0.034; visual mesh filename=../dae/thigh_mirror.dae
- link RL_hip: geometry collision cylinder length=0.04 radius=0.046; visual mesh filename=../dae/hip.dae
- link RL_thigh: geometry collision box size=0.213 0.0245 0.034; visual mesh filename=../dae/thigh.dae
- link RR_hip: geometry collision cylinder length=0.04 radius=0.046; visual mesh filename=../dae/hip.dae
- link RR_thigh: geometry collision box size=0.213 0.0245 0.034; visual mesh filename=../dae/thigh_mirror.dae
- link base: geometry collision box size=0.3762 0.0935 0.114; visual mesh filename=../dae/base.dae
Joints:
- added joint FL_calf_rotor_joint: type fixed, parent FL_thigh, child FL_calf_rotor, origin xyz=0 -0.03235 0 rpy=0 0 0
- added joint FL_hip_rotor_joint: type fixed, parent base, child FL_hip_rotor, origin xyz=0.11215 0.04675 0 rpy=0 0 0
- added joint FL_thigh_rotor_joint: type fixed, parent FL_hip, child FL_thigh_rotor, origin xyz=0 -0.00015 0 rpy=0 0 0
- added joint FR_calf_rotor_joint: type fixed, parent FR_thigh, child FR_calf_rotor, origin xyz=0 0.03235 0 rpy=0 0 0
- added joint FR_hip_rotor_joint: type fixed, parent base, child FR_hip_rotor, origin xyz=0.11215 -0.04675 0 rpy=0 0 0
- added joint FR_thigh_rotor_joint: type fixed, parent FR_hip, child FR_thigh_rotor, origin xyz=0 0.00015 0 rpy=0 0 0
- added joint RL_calf_rotor_joint: type fixed, parent RL_thigh, child RL_calf_rotor, origin xyz=0 -0.03235 0 rpy=0 0 0
- added joint RL_hip_rotor_joint: type fixed, parent base, child RL_hip_rotor, origin xyz=-0.11215 0.04675 0 rpy=0 0 0
- added joint RL_thigh_rotor_joint: type fixed, parent RL_hip, child RL_thigh_rotor, origin xyz=0 -0.00015 0 rpy=0 0 0
- added joint RR_calf_rotor_joint: type fixed, parent RR_thigh, child RR_calf_rotor, origin xyz=0 0.03235 0 rpy=0 0 0
- added joint RR_hip_rotor_joint: type fixed, parent base, child RR_hip_rotor, origin xyz=-0.11215 -0.04675 0 rpy=0 0 0
- added joint RR_thigh_rotor_joint: type fixed, parent RR_hip, child RR_thigh_rotor, origin xyz=0 0.00015 0 rpy=0 0 0
- added joint front_camera_joint: type fixed, parent base, child front_camera, origin xyz=0.32715 -0.00003 0.04297 rpy=0 0 0
- joint FL_calf_joint: limit lower=-2.7227 upper=-0.83776 effort=45.43 velocity=15.7 -> lower=-2.7227 upper=-0.83776 effort=45.43 velocity=15.70
- joint FR_calf_joint: limit lower=-2.7227 upper=-0.83776 effort=45.43 velocity=15.7 -> lower=-2.7227 upper=-0.83776 effort=45.43 velocity=15.70
- joint RL_calf_joint: limit lower=-2.7227 upper=-0.83776 effort=45.43 velocity=15.7 -> lower=-2.7227 upper=-0.83776 effort=45.43 velocity=15.70
- joint RR_calf_joint: limit lower=-2.7227 upper=-0.83776 effort=45.43 velocity=15.7 -> lower=-2.7227 upper=-0.83776 effort=45.43 velocity=15.70
